File: PROYECTOO.sch (EAGLE design)
At the start: 59 parts, among them IC1 AD8226ARZ, IC10 ESP32-S3-WROOM-1-N16R8, IC11 LMV321AIDCKR, IC2 LMV321AIDCKR, IC3 LMV321AIDCKR, IC4 LP38692MP-3.3_NOPB, IC5 LMV321AIDCKR, IC6 MCP73831T-2ACI_OT, IC7 LMV321AIDCKR, IC8 LMV321AIDCKR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

Commit message: Add files via upload
Other:
- note added: "CARGA"
- note added: "ESP32"
- note added: "FILTRO PASA BANDA"
- note added: "PANTALLA"
- note added: "REGULADOR 3.3V"
- note added: "VOLTAJE REF"
Changed lines of the file:
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@@
 <wire x1="436.88" y1="99.06" x2="436.88" y2="66.04" width="0.1524" layer="94" style="shortdash"/>
 <wire x1="436.88" y1="66.04" x2="398.78" y2="66.04" width="0.1524" layer="94" style="shortdash"/>
+<text x="88.9" y="124.46" size="1.778" layer="94">FILTRO PASA BANDA</text>
+<text x="66.04" y="106.68" size="1.778" layer="94" rot="R180">CARGA</text>
+<text x="50.8" y="38.1" size="1.778" layer="94" rot="R180">REGULADOR 3.3V</text>
+<text x="355.6" y="124.46" size="1.778" layer="94" rot="R180">ESP32</text>
+<text x="421.64" y="93.98" size="1.778" layer="94" rot="R180">PANTALLA</text>
+<text x="111.76" y="60.96" size="1.778" layer="94" rot="R180">VOLTAJE REF</text>
 </plain>
 <instances>
