File: PROYECTOO.sch (EAGLE design)
At the start: 37 parts, among them IC1 AD8226ARZ, IC10 ESP32-S3-WROOM-1-N16R8, IC11 LMV321AIDCKR, IC2 LMV321AIDCKR, IC3 LMV321AIDCKR, IC4 LP38692MP-3.3_NOPB, IC6 MCP73831T-2ACI_OT, J1 204926-1103, J2 SJ-3523-SMT-TR

Commit message: Add files via upload
Parts:
- removed C13, C14: 10v, capacitor-wima:C2,5-3
- removed G1: AB9V, battery:AB9V
- removed LED2: LAP4-BOTTOM, led:LAP4-BOTTOM
- removed R11: 12K, resistor-shunt:SMK
- removed R12: 1k, resistor-shunt:SMK
- removed R15: 220, rcl:R-EU_0204/2V
- removed R16: 2k, rcl:R-EU_0204/2V
- removed RG: 50, resistor-shunt:SMK
- removed SV1: (no value), con-lstb:MA04-1
- removed SW1: (no value), special:SW_DIP-1
- added C10, C9: (no value), rcl:C-EUC0805
- added CHARGING: (no value), led:LEDCHIP-LED0805
- added J3: 1769, 1769:1769
- added OLED: (no value), con-lstb:MA04-1
- added R13, R4, R5, R8, R9: (no value), rcl:R-EU_R0805
- added S3: SS4-CM-V-T_R, SS4-CM-V-T_R:SS4-CM-V-T_R
- C1, C2, C4, C5: value 1u -> (none); device rcl:C-EUC0402K -> rcl:C-EUC0805
- C3: value 10u -> (none); device rcl:C-EUC0402K -> rcl:C-EUC0805
- C6, C7, C8: device capacitor-wima:C2.5/2 -> rcl:C-EUC0805
- J1: value 204926-1103 -> USB3500-30-A-KIT; device 204926-1103:204926-1103 -> USB3500-30-A-KIT:USB3500-30-A-KIT
- R1, R3: value 1.6k -> (none); device rcl:R-EU_0204/2V -> rcl:R-EU_R0805
- R10: value 12K -> (none); device resistor-shunt:SMK -> rcl:R-EU_R0805
- R2: value 10K -> (none); device resistor-shunt:SMK -> rcl:R-EU_R0805
- R6, R7: value 320k -> (none); device rcl:R-EU_0204/2V -> rcl:R-EU_R0805
Connections:
- removed net N$13: IC3.-IN, IC3.OUT, R7.1
- removed net N$24: IC6.STAT, R15.1
- removed net N$25: LED2.C, R15.2
- removed net N$27: IC6.PROG, R16.2
- removed net N$46: IC11.OUT, R2.1
- removed net OUT_1: IC1.VOUT, R1.2
- removed net VCC: C14.1, C3.1, C6.2, IC1.+VS, IC10.3V3, IC11.V+, IC2.V+, IC3.V+, IC4.OUT, IC6.VDD, J1.VBUS, LED2.A, PS1.EN, PS1.VIN, R10.2, R11.2, SV1.2
- new net +3V3: C3.1, C6.2, IC1.+VS, IC10.3V3, IC11.V+, IC2.V+, IC3.V+, IC4.OUT, OLED.2, PS1.EN, PS1.VIN, R10.2, R8.2
- new net +5V: C5.2, CHARGING.A, IC6.VDD, J1.1, S3.NO_1
- new net +D: IC10.IO20, J1.3
- new net -D: IC10.IO19, J1.2
- new net BATT: C10.2, IC6.VBAT, J3.1
- new net DAC1: IC10.IO17
- new net DAC2: IC10.IO18
- new net FLASH: C8.2, S2.NO_1
- new net IRQ_RA02: IC10.IO16
- new net LED1: IC10.IO21
- new net LED2: IC10.IO14
- new net LED3: IC10.IO13
- new net MISO: IC10.IO39
- new net MOSI: IC10.IO1
- new net N$1: IC1.RG_1, R1.2
- new net N$10: IC6.PROG, R7.2
- new net N$20: IC10.TXD0
- new net NSS: IC10.IO37
- new net OUT1: IC1.VOUT, R13.1
- new net RESET: C7.2, IC10.EN, R8.1, S1.NO_1
- new net RST_RA: IC10.IO35
- new net RX: IC10.RXD0
- new net SCK: IC10.IO38
- new net TOUCHPAD1: IC10.IO9
- new net TOUCHPAD2: IC10.IO10
- new net TOUCHPAD3: IC10.IO11
- new net VOUT1: IC11.+IN, IC3.-IN, IC3.OUT, R4.2
- new net VOUT2: IC10.IO7, IC11.OUT, R6.1
- net +BATT: now also S3.NC; no longer C13.1, G1.+, IC6.VBAT, SW1.2
- net GND: now also C1.1, C10.1, C5.1, J1.5, J3.2, OLED.1, R7.1, R9.1; no longer C1.2, C13.2, C14.2, C8.2, G1.-, J1.GND, J1.MH5, J1.MH6, R16.1, R6.2, S2.NO_1, SV1.1
- net N$11: now also C4.1, C9.2, R4.1; no longer C4.2, C5.1, R7.2
- net N$12: now also C4.2, R9.2; no longer C5.2, R6.1
- net N$19: now also S3.COM; no longer SW1.1
- net N$3: now also IC1.RG_2, R1.1; no longer IC1.RG_1, RG.1
- net N$4: now also IC6.STAT, R2.1; no longer IC1.RG_2, RG.2
- net N$43: now also R10.1; no longer R11.1
- net N$44: now also R5.2, R6.2; no longer R12.1, R2.2
- net N$5: now also C1.2; no longer C1.1
- net N$6: now also R13.2; no longer R1.1
- net N$8: now also CHARGING.C, R2.2; no longer C7.2, IC10.EN, R10.1, S1.NO_1
- net N$9: now also C9.1; no longer C4.1
- net SCL: now also IC10.IO2, OLED.3; no longer IC10.RXD0, SV1.3
- net SDA: now also IC10.IO41, OLED.4; no longer IC10.IO40, SV1.4
- net VSS: now also J2.SLEEVE, R5.1; no longer IC11.+IN
Other:
- moved on the sheet: C1, C3, C4, C5, C6, C7, C8, IC10, R1, R10, R2, R6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
