File: PROYECTOO.brd (EAGLE design)
At the start: 160 x 100 mm, 37 parts, among them IC1 AD8226ARZ, IC10 ESP32-S3-WROOM-1-N16R8, IC11 LMV321AIDCKR, IC2 LMV321AIDCKR, IC3 LMV321AIDCKR, IC4 LP38692MP-3.3_NOPB, IC6 MCP73831T-2ACI_OT, J1 204926-1103, J2 SJ-3523-SMT-TR

Commit message: Add files via upload
Parts:
- removed C13, C14: 10v, capacitor-wima:C2.5-3
- removed G1: AB9V, battery:AB9V
- removed LED2: LAP4-BOTTOM, led:P47F-BOTTOM
- removed R11: 12K, resistor-shunt:SMK
- removed R12: 1k, resistor-shunt:SMK
- removed R15: 220, rcl:0204V
- removed R16: 2k, rcl:0204V
- removed RG: 50, resistor-shunt:SMK
- removed SV1: (no value), con-lstb:MA04-1
- removed SW1: (no value), special:EDG-01
- added C10, C9: (no value), rcl:C0805
- added CHARGING: (no value), led:CHIP-LED0805
- added J3: 1769, 1769:1769
- added OLED: (no value), con-lstb:MA04-1
- added R13, R4, R5, R8, R9: (no value), rcl:R0805
- added S3: SS4-CM-V-T_R, SS4-CM-V-T_R:SS4CMVTR
- C1, C2, C4, C5: value 1u -> (none); device rcl:C0402K -> rcl:C0805
- C3: value 10u -> (none); device rcl:C0402K -> rcl:C0805
- C6, C7, C8: device capacitor-wima:C2.5-2 -> rcl:C0805
- J1: value 204926-1103 -> USB3500-30-A-KIT; device 204926-1103:2049261103 -> USB3500-30-A-KIT:USB350030AKIT
- R1, R3: value 1.6k -> (none); device rcl:0204V -> rcl:R0805
- R10: value 12K -> (none); device resistor-shunt:SMK -> rcl:R0805
- R2: value 10K -> (none); device resistor-shunt:SMK -> rcl:R0805
- R6, R7: value 320k -> (none); device rcl:0204V -> rcl:R0805
- moved R2 107.2 mm to (39.4, 16.5)
- moved IC4 104.2 mm to (53.8, 22.1), turned to 90 degrees
- moved PS1 99.5 mm to (38.7, 27.9), turned to 90 degrees
- moved IC2 94.6 mm to (15.9, 31.1)
- moved C3 94.1 mm to (16.5, 24.8), turned to 270 degrees
- moved S1 93.6 mm to (24.8, 64.1)
- moved IC11 91.5 mm to (34.9, 22.9)
- moved C1 90.4 mm to (12.7, 35.6)
- moved J1 89.2 mm to (53.3, 3.81)
- moved R10 84.5 mm to (15.9, 52.1), turned to 180 degrees
- moved IC6 82.9 mm to (27.0, 12.7), turned to 180 degrees
- moved IC10 82.9 mm to (45.7, 57.8), turned to 270 degrees
- moved C8 80.2 mm to (15.2, 57.1)
- moved C7 74.9 mm to (15.2, 62.2), turned to 180 degrees
- moved C5 70.5 mm to (21.0, 13.3), turned to 270 degrees
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Connections:
- removed net N$13: IC3.3, IC3.4, R7.1
- removed net N$24: IC6.1, R15.1
- removed net N$25: LED2.C, R15.2
- removed net N$27: IC6.5, R16.2
- removed net N$46: IC11.4, R2.1
- removed net OUT_1: IC1.7, R1.2
- removed net VCC: C14.1, C3.1, C6.2, IC1.8, IC10.2, IC11.5, IC2.5, IC3.5, IC4.3, IC6.4, J1.1, LED2.A, PS1.3, PS1.4, R10.2, R11.2, SV1.2
- new net +3V3: C3.1, C6.2, IC1.8, IC10.2, IC11.5, IC2.5, IC3.5, IC4.3, OLED.2, PS1.3, PS1.4, R10.2, R8.2
- new net +5V: C5.2, CHARGING.A, IC6.4, J1.1, S3.A1
- new net +D: IC10.14, J1.3
- new net -D: IC10.13, J1.2
- new net BATT: C10.2, IC6.3, J3.1
- new net DAC1: IC10.10
- new net DAC2: IC10.11
- new net FLASH: C8.2, S2.1
- new net IRQ_RA02: IC10.9
- new net LED1: IC10.23
- new net LED2: IC10.22
- new net LED3: IC10.21
- new net MISO: IC10.32
- new net MOSI: IC10.39
- new net N$1: IC1.2, R1.2
- new net N$10: IC6.5, R7.2
- new net N$20: IC10.37
- new net NSS: IC10.30
- new net OUT1: IC1.7, R13.1
- new net RESET: C7.2, IC10.3, R8.1, S1.1
- new net RST_RA: IC10.28
- new net RX: IC10.36
- new net SCK: IC10.31
- new net TOUCHPAD1: IC10.17
- new net TOUCHPAD2: IC10.18
- new net TOUCHPAD3: IC10.19
- new net VOUT1: IC11.1, IC3.3, IC3.4, R4.2
- new net VOUT2: IC10.7, IC11.4, R6.1
- net +BATT: now also S3.B1; no longer C13.1, G1.+, IC6.3, SW1.2
- net GND: now also C1.1, C10.1, C5.1, J3.2, OLED.1, R7.1, R9.1; no longer C1.2, C13.2, C14.2, C8.2, G1.-, J1.MH5, J1.MH6, R16.1, R6.2, S2.1, SV1.1
- net N$11: now also C4.1, C9.2, R4.1; no longer C4.2, C5.1, R7.2
- net N$12: now also C4.2, R9.2; no longer C5.2, R6.1
- net N$19: now also S3.C1; no longer SW1.1
- net N$3: now also IC1.3, R1.1; no longer IC1.2, RG.1
- net N$4: now also IC6.1, R2.1; no longer IC1.3, RG.2
- net N$43: now also R10.1; no longer R11.1
- net N$44: now also R5.2, R6.2; no longer R12.1, R2.2
- net N$5: now also C1.2; no longer C1.1
- net N$6: now also R13.2; no longer R1.1
- net N$8: now also CHARGING.C, R2.2; no longer C7.2, IC10.3, R10.1, S1.1
- net N$9: now also C9.1; no longer C4.1
- net SCL: now also IC10.38, OLED.3; no longer IC10.36, SV1.3
- net SDA: now also IC10.34, OLED.4; no longer IC10.33, SV1.4
- net VSS: now also J2.1, R5.1; no longer IC11.1
Routing:
- net +3V3: track 0.00 -> 192.4 mm, vias 0 -> 8
- net VOUT2: track 0.00 -> 127.3 mm, vias 0 -> 4
- net +D: track 0.00 -> 74.6 mm, vias 0 -> 2
- net -D: track 0.00 -> 71.6 mm, vias 0 -> 2
- net VSS: track 0.00 -> 60.3 mm, vias 0 -> 2
- net +5V: track 0.00 -> 54.0 mm, vias 0 -> 4
- net SCL: track 0.00 -> 52.5 mm, vias 0 -> 2
- net N$10: track 0.00 -> 49.8 mm
- net N$19: track 0.00 -> 46.5 mm
- net RESET: track 0.00 -> 45.3 mm
- net SDA: track 0.00 -> 40.6 mm, vias 0 -> 2
- net N$2: track 0.00 -> 28.8 mm
- net N$43: track 0.00 -> 25.5 mm
- net N$44: track 0.00 -> 21.7 mm, vias 0 -> 2
- net N$17: track 0.00 -> 18.6 mm
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Other:
- board size 160 x 100 mm -> 60.6 x 80 mm
